Commit message: added correct workfolder and instructions showing commands to remember for usage of mikibot

File: miki_ws/src/my_mikibot/urdf/mikibot.urdf (robot description, URDF)
Before this commit: robot henpai, 9 links, 8 joints
Links:
- link base: mass None -> 10
- link bl_wheel: mass None -> 10
- link body: mass None -> 10
- link br_wheel: mass None -> 10
- link rightman: mass None -> 10
Joints:
- joint RWb_joint: axis (none) -> 0 0 1
- joint lWb_joint: axis (none) -> 0 0 1

Commit message: added collision to robot

File: miki_ws/src/my_mikibot/urdf/mikibot.urdf (robot description, URDF)
Before this commit: robot mikibot, 9 links, 8 joints
Links:
- link base: geometry collision box size=0.6 0.5 0.1; visual box size=0.6 0.5 0.1
- link bl_wheel: geometry collision cylinder length=0.1 radius=0.05; visual cylinder length=0.1 radius=0.05
- link body: geometry collision cylinder length=0.1 radius=0.4; visual cylinder length=0.1 radius=0.4
- link br_wheel: geometry collision cylinder length=0.1 radius=0.05; visual cylinder length=0.1 radius=0.05
- link lefthan: geometry collision box size=0.4 0.02 0.05; visual box size=0.4 0.02 0.05
- link leftman: geometry collision sphere length=0.1 radius=0.05; visual cylinder length=0.1 radius=0.05
- link righthan: geometry collision box size=0.4 0.02 0.05; visual box size=0.4 0.02 0.05
- link rightman: geometry collision cylinder length=0.1 radius=0.05; visual cylinder length=0.1 radius=0.05
- link roller: geometry collision sphere length=0.1 radius=0.06; visual sphere length=0.1 radius=0.06

Commit message: added missing colissions

File: miki_ws/src/my_mikibot/urdf/mikibot.urdf (robot description, URDF)
Before this commit: robot mikibot, 9 links, 8 joints
Links:
- link lefthan: mass None -> 10
- link leftman: mass None -> 10
- link roller: mass None -> 10

Commit message: fixed urdf conflicts and added new launch parameters

File: miki_ws/src/my_mikibot/urdf/mikibot.urdf (robot description, URDF)
Before this commit: robot mikibot, 9 links, 8 joints
Links:
- link righthan: mass None -> 10
Joints:
- removed joint left_mandible
- added joint Left_mandible: type revolute, parent body, child leftman, origin xyz=0 0 0 rpy=0 0 0, axis 0 0 -1, limit lower=0.0 upper=0.548 effort=1000.0 velocity=0.5

Commit message: fixed steering

File: miki_ws/src/my_mikibot/urdf/mikibot.urdf (robot description, URDF)
Before this commit: robot mikibot, 9 links, 8 joints
Links:
- removed link base
- removed link lefthan
- removed link righthan
- added link base_footprint, mass 10; collision box size=0.2 0.3 0.1; visual box size=0.2 0.3 0.1
- added link lefthand, mass 10; collision box size=0.4 0.02 0.05; visual box size=0.3 0.02 0.05
- added link righthand, mass 10; collision box size=0.4 0.02 0.05; visual box size=0.3 0.02 0.05
- link bl_wheel: geometry collision cylinder length=0.05 radius=0.04; visual cylinder length=0.05 radius=0.04
- link body: geometry collision cylinder length=0.1 radius=0.2; visual cylinder length=0.1 radius=0.2
- link br_wheel: geometry collision cylinder length=0.05 radius=0.04; visual cylinder length=0.05 radius=0.04
- link leftman: geometry collision sphere length=0.1 radius=0.03; visual cylinder length=0.1 radius=0.03
- link rightman: geometry collision cylinder length=0.1 radius=0.03; visual cylinder length=0.1 radius=0.03
Joints:
- removed joint RWb_joint
- removed joint lWb_joint
- added joint lwd_joint: type continuous, parent base_footprint, child bl_wheel, origin xyz=-0.1 0.1 -0.05 rpy=1.57075 0 3.14, axis 0 0 1, limit effort=100 velocity=100
- added joint rwd_joint: type continuous, parent base_footprint, child br_wheel, origin xyz=-0.1 -0.1 -0.05 rpy=1.57075 0 3.14, axis 0 0 1, limit effort=100 velocity=100
- joint Left_mandible: parent body -> base_footprint
- joint Right_mandible: parent body -> base_footprint
- joint base_to_body: parent base -> base_footprint
- joint gripper_left: child lefthan -> lefthand; parent leftman -> base_footprint
- joint gripper_right: child righthan -> righthand; parent rightman -> base_footprint
- joint rollercast: origin xyz=0.2 0 -0.05 rpy=0 0 0 -> xyz=0.1 0 -0.025 rpy=0 0 0; parent base -> base_footprint

Commit message: fixed joint state publisher

File: miki_ws/src/my_mikibot/urdf/mikibot.urdf (robot description, URDF)
Before this commit: robot mikibot, 9 links, 8 joints
Links:
- removed link base_footprint
- added link base, mass 10; collision box size=0.2 0.3 0.1; visual box size=0.2 0.3 0.1
- added link fbump, mass 10; collision box size=0.2 0.2 0.02; visual box size=0.2 0.2 0.02
Joints:
- added joint bumpbod: type fixed, parent base, child fbump, origin xyz=0 0 0
- joint Left_mandible: parent base_footprint -> base; type revolute -> fixed
- joint Right_mandible: parent base_footprint -> base; type revolute -> fixed
- joint base_to_body: parent base_footprint -> base
- joint gripper_left: axis (none) -> 0 0 1; limit (none) -> lower=0.0 upper=-0.548 effort=1000.0 velocity=0.5; origin xyz=0 0 0 -> xyz=0 0 0 rpy=0 0 0; parent base_footprint -> base; type fixed -> revolute
- joint gripper_right: axis (none) -> 0 0 1; limit (none) -> lower=0.0 upper=0.548 effort=1000.0 velocity=0.5; origin xyz=0 0 0 -> xyz=0 0 0 rpy=0 0 0; parent base_footprint -> base; type fixed -> revolute
- joint lwd_joint: parent base_footprint -> base
- joint rollercast: parent base_footprint -> base
- joint rwd_joint: parent base_footprint -> base
